File: layout-pcb/keyboard.kicad_pcb (KiCad board)
At the start: 6 copper layers, 374.7 x 131.8 mm, 276 parts

Commit message: pcb basic wiring
Parts:
- moved D78 0.35 mm to (323.1, 126.0)
- moved D79 0.35 mm to (342.1, 126.0)
Connections:
- D14 pad 2: unconnected-(D14-DOUT-Pad2) -> 14p2-32p4
- D32 pad 2: unconnected-(D32-DOUT-Pad2) -> Net-(D32-DOUT)
- D32 pad 4: unconnected-(D32-DIN-Pad4) -> 14p2-32p4
- D33 pad 2: unconnected-(D33-DOUT-Pad2) -> Net-(D33-DOUT)
- D33 pad 4: unconnected-(D33-DIN-Pad4) -> Net-(D32-DOUT)
- D34 pad 2: unconnected-(D34-DOUT-Pad2) -> Net-(D34-DOUT)
- D34 pad 4: unconnected-(D34-DIN-Pad4) -> Net-(D33-DOUT)
- D35 pad 2: unconnected-(D35-DOUT-Pad2) -> Net-(D35-DOUT)
- D35 pad 4: unconnected-(D35-DIN-Pad4) -> Net-(D34-DOUT)
- D36 pad 2: unconnected-(D36-DOUT-Pad2) -> Net-(D36-DOUT)
- D36 pad 4: unconnected-(D36-DIN-Pad4) -> Net-(D35-DOUT)
- D37 pad 2: unconnected-(D37-DOUT-Pad2) -> Net-(D37-DOUT)
- D37 pad 4: unconnected-(D37-DIN-Pad4) -> Net-(D36-DOUT)
- D38 pad 2: unconnected-(D38-DOUT-Pad2) -> Net-(D38-DOUT)
- D38 pad 4: unconnected-(D38-DIN-Pad4) -> Net-(D37-DOUT)
- D39 pad 2: unconnected-(D39-DOUT-Pad2) -> 39p2-40p4
- D39 pad 4: unconnected-(D39-DIN-Pad4) -> Net-(D38-DOUT)
- D40 pad 2: unconnected-(D40-DOUT-Pad2) -> Net-(D40-DOUT)
- D40 pad 4: unconnected-(D40-DIN-Pad4) -> 39p2-40p4
- D41 pad 2: unconnected-(D41-DOUT-Pad2) -> Net-(D41-DOUT)
- D41 pad 4: unconnected-(D41-DIN-Pad4) -> Net-(D40-DOUT)
- D42 pad 2: unconnected-(D42-DOUT-Pad2) -> Net-(D42-DOUT)
- D42 pad 4: unconnected-(D42-DIN-Pad4) -> Net-(D41-DOUT)
- D43 pad 2: unconnected-(D43-DOUT-Pad2) -> Net-(D43-DOUT)
- D43 pad 4: unconnected-(D43-DIN-Pad4) -> Net-(D42-DOUT)
- D44 pad 2: unconnected-(D44-DOUT-Pad2) -> Net-(D44-DOUT)
- D44 pad 4: unconnected-(D44-DIN-Pad4) -> Net-(D43-DOUT)
- D45 pad 2: unconnected-(D45-DOUT-Pad2) -> Net-(D45-DOUT)
- D45 pad 4: unconnected-(D45-DIN-Pad4) -> Net-(D44-DOUT)
- D46 pad 2: unconnected-(D46-DOUT-Pad2) -> Net-(D46-DOUT)
- D46 pad 4: unconnected-(D46-DIN-Pad4) -> Net-(D45-DOUT)
- D47 pad 2: unconnected-(D47-DOUT-Pad2) -> Net-(D47-DOUT)
- D47 pad 4: unconnected-(D47-DIN-Pad4) -> Net-(D46-DOUT)
- D48 pad 2: unconnected-(D48-DOUT-Pad2) -> Net-(D48-DOUT)
- D48 pad 4: unconnected-(D48-DIN-Pad4) -> Net-(D47-DOUT)
- D49 pad 2: unconnected-(D49-DOUT-Pad2) -> 49p2-65p4
- D49 pad 4: unconnected-(D49-DIN-Pad4) -> Net-(D48-DOUT)
- D50 pad 2: unconnected-(D50-DOUT-Pad2) -> 50p2-66p4
- D50 pad 4: unconnected-(D50-DIN-Pad4) -> Net-(D50-DIN)
- D51 pad 2: unconnected-(D51-DOUT-Pad2) -> Net-(D50-DIN)
- D51 pad 4: unconnected-(D51-DIN-Pad4) -> Net-(D51-DIN)
- D52 pad 2: unconnected-(D52-DOUT-Pad2) -> Net-(D51-DIN)
- D52 pad 4: unconnected-(D52-DIN-Pad4) -> 53p2-52p4
- D53 pad 2: unconnected-(D53-DOUT-Pad2) -> 53p2-52p4
- D53 pad 4: unconnected-(D53-DIN-Pad4) -> Net-(D53-DIN)
- D54 pad 2: unconnected-(D54-DOUT-Pad2) -> Net-(D53-DIN)
- D54 pad 4: unconnected-(D54-DIN-Pad4) -> Net-(D54-DIN)
- D55 pad 2: unconnected-(D55-DOUT-Pad2) -> Net-(D54-DIN)
- D55 pad 4: unconnected-(D55-DIN-Pad4) -> Net-(D55-DIN)
- D56 pad 2: unconnected-(D56-DOUT-Pad2) -> Net-(D55-DIN)
- D56 pad 4: unconnected-(D56-DIN-Pad4) -> Net-(D56-DIN)
- D57 pad 2: unconnected-(D57-DOUT-Pad2) -> Net-(D56-DIN)
- D57 pad 4: unconnected-(D57-DIN-Pad4) -> Net-(D57-DIN)
- D58 pad 2: unconnected-(D58-DOUT-Pad2) -> Net-(D57-DIN)
- D58 pad 4: unconnected-(D58-DIN-Pad4) -> Net-(D58-DIN)
- D59 pad 2: unconnected-(D59-DOUT-Pad2) -> Net-(D58-DIN)
- D59 pad 4: unconnected-(D59-DIN-Pad4) -> Net-(D59-DIN)
- D60 pad 2: unconnected-(D60-DOUT-Pad2) -> Net-(D59-DIN)
- D60 pad 4: unconnected-(D60-DIN-Pad4) -> Net-(D60-DIN)
- D61 pad 2: unconnected-(D61-DOUT-Pad2) -> Net-(D60-DIN)
- D61 pad 4: unconnected-(D61-DIN-Pad4) -> Net-(D61-DIN)
- D62 pad 2: unconnected-(D62-DOUT-Pad2) -> Net-(D61-DIN)
- D62 pad 4: unconnected-(D62-DIN-Pad4) -> Net-(D62-DIN)
- D63 pad 2: unconnected-(D63-DOUT-Pad2) -> Net-(D62-DIN)
- D63 pad 4: unconnected-(D63-DIN-Pad4) -> Net-(D63-DIN)
- D64 pad 2: unconnected-(D64-DOUT-Pad2) -> Net-(D63-DIN)
- D64 pad 4: unconnected-(D64-DIN-Pad4) -> Net-(D64-DIN)
- D65 pad 2: unconnected-(D65-DOUT-Pad2) -> Net-(D64-DIN)
- D65 pad 4: unconnected-(D65-DIN-Pad4) -> 49p2-65p4
- D66 pad 2: unconnected-(D66-DOUT-Pad2) -> Net-(D66-DOUT)
- D66 pad 4: unconnected-(D66-DIN-Pad4) -> 50p2-66p4
- D67 pad 2: unconnected-(D67-DOUT-Pad2) -> Net-(D67-DOUT)
- D67 pad 4: unconnected-(D67-DIN-Pad4) -> Net-(D66-DOUT)
- D68 pad 2: unconnected-(D68-DOUT-Pad2) -> Net-(D68-DOUT)
- D68 pad 4: unconnected-(D68-DIN-Pad4) -> Net-(D67-DOUT)
- D69 pad 2: unconnected-(D69-DOUT-Pad2) -> Net-(D69-DOUT)
- D69 pad 4: unconnected-(D69-DIN-Pad4) -> Net-(D68-DOUT)
- D70 pad 2: unconnected-(D70-DOUT-Pad2) -> Net-(D70-DOUT)
- D70 pad 4: unconnected-(D70-DIN-Pad4) -> Net-(D69-DOUT)
- D71 pad 2: unconnected-(D71-DOUT-Pad2) -> Net-(D71-DOUT)
- D71 pad 4: unconnected-(D71-DIN-Pad4) -> Net-(D70-DOUT)
- D72 pad 2: unconnected-(D72-DOUT-Pad2) -> Net-(D72-DOUT)
- D72 pad 4: unconnected-(D72-DIN-Pad4) -> Net-(D71-DOUT)
- D73 pad 2: unconnected-(D73-DOUT-Pad2) -> Net-(D73-DOUT)
- D73 pad 4: unconnected-(D73-DIN-Pad4) -> Net-(D72-DOUT)
- D74 pad 2: unconnected-(D74-DOUT-Pad2) -> Net-(D74-DOUT)
- D74 pad 4: unconnected-(D74-DIN-Pad4) -> Net-(D73-DOUT)
- D75 pad 2: unconnected-(D75-DOUT-Pad2) -> Net-(D75-DOUT)
- D75 pad 4: unconnected-(D75-DIN-Pad4) -> Net-(D74-DOUT)
- D76 pad 2: unconnected-(D76-DOUT-Pad2) -> Net-(D76-DOUT)
- D76 pad 4: unconnected-(D76-DIN-Pad4) -> Net-(D75-DOUT)
- D77 pad 2: unconnected-(D77-DOUT-Pad2) -> Net-(D77-DOUT)
- D77 pad 4: unconnected-(D77-DIN-Pad4) -> Net-(D76-DOUT)
- D78 pad 2: unconnected-(D78-DOUT-Pad2) -> 78p2-79p4
- D78 pad 4: unconnected-(D78-DIN-Pad4) -> Net-(D77-DOUT)
- D79 pad 2: unconnected-(D79-DOUT-Pad2) -> Net-(D79-DOUT)
- D79 pad 4: unconnected-(D79-DIN-Pad4) -> 78p2-79p4
- D80 pad 2: unconnected-(D80-DOUT-Pad2) -> Net-(D80-DOUT)
- D80 pad 4: unconnected-(D80-DIN-Pad4) -> Net-(D79-DOUT)
- D81 pad 2: unconnected-(D81-DOUT-Pad2) -> 81p2-91p4
- D81 pad 4: unconnected-(D81-DIN-Pad4) -> Net-(D80-DOUT)
- D82 pad 4: unconnected-(D82-DIN-Pad4) -> Net-(D82-DIN)
- D83 pad 2: unconnected-(D83-DOUT-Pad2) -> Net-(D82-DIN)
- D83 pad 4: unconnected-(D83-DIN-Pad4) -> Net-(D83-DIN)
- D84 pad 2: unconnected-(D84-DOUT-Pad2) -> Net-(D83-DIN)
- D84 pad 4: unconnected-(D84-DIN-Pad4) -> Net-(D84-DIN)
- D85 pad 2: unconnected-(D85-DOUT-Pad2) -> Net-(D84-DIN)
- D85 pad 4: unconnected-(D85-DIN-Pad4) -> Net-(D85-DIN)
- D86 pad 2: unconnected-(D86-DOUT-Pad2) -> Net-(D85-DIN)
- D86 pad 4: unconnected-(D86-DIN-Pad4) -> Net-(D86-DIN)
- D87 pad 2: unconnected-(D87-DOUT-Pad2) -> Net-(D86-DIN)
- D87 pad 4: unconnected-(D87-DIN-Pad4) -> Net-(D87-DIN)
- D88 pad 2: unconnected-(D88-DOUT-Pad2) -> Net-(D87-DIN)
- D88 pad 4: unconnected-(D88-DIN-Pad4) -> Net-(D88-DIN)
- D89 pad 2: unconnected-(D89-DOUT-Pad2) -> Net-(D88-DIN)
- D89 pad 4: unconnected-(D89-DIN-Pad4) -> Net-(D89-DIN)
- D90 pad 2: unconnected-(D90-DOUT-Pad2) -> Net-(D89-DIN)
- D90 pad 4: unconnected-(D90-DIN-Pad4) -> Net-(D90-DIN)
- D91 pad 2: unconnected-(D91-DOUT-Pad2) -> Net-(D90-DIN)
- D91 pad 4: unconnected-(D91-DIN-Pad4) -> 81p2-91p4
- D92 pad 2: unconnected-(D92-DOUT-Pad2) -> Net-(D92-DOUT)
- D92 pad 4: unconnected-(D92-DIN-Pad4) -> LED-Status IN
- D93 pad 2: unconnected-(D93-DOUT-Pad2) -> Net-(D93-DOUT)
- D93 pad 4: unconnected-(D93-DIN-Pad4) -> Net-(D92-DOUT)
- D94 pad 4: unconnected-(D94-DIN-Pad4) -> Net-(D93-DOUT)
Routing:
- net row4: track 0.00 -> 333.3 mm
- net row5: track 0.00 -> 325.5 mm
- net row3: track 0.00 -> 317.0 mm
- net row0: track 0.00 -> 268.7 mm
- net LED_GND: track 1.10 -> 204.8 mm, vias 0 -> 94
- net LED_PWR: track 26.2 -> 168.5 mm, vias 16 -> 94
- net col13: track 0.00 -> 137.5 mm, vias 0 -> 5
- net col3: track 0.00 -> 136.9 mm, vias 0 -> 6
- net col10: track 0.00 -> 135.7 mm, vias 0 -> 6
- net col11: track 0.00 -> 132.1 mm, vias 0 -> 6
- net col14: track 0.00 -> 121.1 mm, vias 0 -> 4
- net col2: track 0.00 -> 116.4 mm, vias 0 -> 5
- net col7: track 0.00 -> 115.6 mm, vias 0 -> 5
- net col8: track 0.00 -> 113.6 mm, vias 0 -> 5
- net col9: track 0.00 -> 113.5 mm, vias 0 -> 5
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
Commit message: pcb basic wiring
Connections:
- D27 pad 4: 26p4-27p2 -> Net-(D27-DIN)
- D28 pad 2: 26p4-27p2 -> Net-(D27-DIN)
Routing:
- net col15: track 11.1 -> 72.9 mm
- net Net-(D27-DIN): track 0.00 -> 30.7 mm
- net 26p4-27p2: track 56.4 -> 25.8 mm
Other:
- outline, holes or cut-outs redrawn
Changed lines of the file:
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@@
 	(net 209 "LED-Status IN")
 	(net 210 "Net-(D93-DOUT)")
-	(net 211 "unconnected-(D82-DOUT-Pad2)")
-	(net 212 "Net-(D30-DIN)")
-	(net 213 "unconnected-(D94-DOUT-Pad2)")
+	(net 211 "Net-(D27-DIN)")
+	(net 212 "unconnected-(D82-DOUT-Pad2)")
+	(net 213 "Net-(D30-DIN)")
+	(net 214 "unconnected-(D94-DOUT-Pad2)")
 	(footprint "MX_Only:MXOnly-1U-Hotswap"
 		(layer "F.Cu")
@@
 			(size 1.5 0.9)
 			(layers "F.Cu" "F.Paste" "F.Mask")
-			(net 211 "unconnected-(D82-DOUT-Pad2)")
+			(net 212 "unconnected-(D82-DOUT-Pad2)")
 			(pinfunction "DOUT")
 			(pintype "output")
@@
 			(size 1.5 0.9)
 			(layers "F.Cu" "F.Paste" "F.Mask")
-			(net 213 "unconnected-(D94-DOUT-Pad2)")
+			(net 214 "unconnected-(D94-DOUT-Pad2)")
 			(pinfunction "DOUT")
 			(pintype "output")
@@
 			(size 1.5 0.9)
 			(layers "F.Cu" "F.Paste" "F.Mask")
-			(net 212 "Net-(D30-DIN)")
+			(net 213 "Net-(D30-DIN)")
 			(pinfunction "DOUT")
 			(pintype "output")
@@
 			(size 1.5 0.9)
 			(layers "F.Cu" "F.Paste" "F.Mask")
-			(net 143 "26p4-27p2")
+			(net 211 "Net-(D27-DIN)")
 			(pinfunction "DOUT")
 			(pintype "output")
@@
 			(size 1.5 0.9)
 			(layers "F.Cu" "F.Paste" "F.Mask")
-			(net 212 "Net-(D30-DIN)")
+			(net 213 "Net-(D30-DIN)")
 			(pinfunction "DIN")
 			(pintype "input")
@@
 			(size 1.5 0.9)
 			(layers "F.Cu" "F.Paste" "F.Mask")
-			(net 143 "26p4-27p2")
+			(net 211 "Net-(D27-DIN)")
 			(pinfunction "DIN")
 			(pintype "input")
@@
 	)
 	(gr_arc
+		(start 393.4625 145.45)
+		(mid 391.998034 148.985534)
+		(end 388.4625 150.45)
+		(stroke
+			(width 0.2)
+			(type default)
+		)
+		(layer "Edge.Cuts")
+	)
+	(gr_arc
+		(start 23.75 150.45)
+		(mid 20.214466 148.985534)
+		(end 18.75 145.45)
+		(stroke
+			(width 0.2)
+			(type default)
+		)
+		(layer "Edge.Cuts")
+	)
+	(gr_arc
 		(start 18.75 18.625)
 		(mid 18.75 18.625)
@@
 	)
 	(gr_line
-		(start 393.4625 18.625)
-		(end 393.4625 150.45)
+		(start 393.4625 23.625)
+		(end 393.4625 145.45)
 		(stroke
 			(width 0.2)
@@
 		(layer "Edge.Cuts")
 	)
+	(gr_arc
+		(start 18.75 23.625)
+		(mid 20.214466 20.089466)
+		(end 23.75 18.625)
+		(stroke
+			(width 0.2)
+			(type default)
+		)
+		(layer "Edge.Cuts")
+	)
 	(gr_line
-		(start 18.75 18.625)
-		(end 393.4625 18.625)
+		(start 23.75 18.625)
+		(end 388.4625 18.625)
 		(stroke
 			(width 0.2)
@@
 	)
 	(gr_line
-		(start 393.4625 150.45)
-		(end 18.75 150.45)
+		(start 388.4625 150.45)
+		(end 23.75 150.45)
 		(stroke
 			(width 0.2)
@@
 	)
 	(gr_line
-		(start 18.75 150.45)
-		(end 18.75 18.625)
+		(start 18.75 145.45)
+		(end 18.75 23.625)
 		(stroke
 			(width 0.2)
@@
 		(layer "Edge.Cuts")
 	)
+	(gr_arc
+		(start 388.4625 18.625)
+		(mid 391.998034 20.089466)
+		(end 393.4625 23.625)
+		(stroke
+			(width 0.2)
+			(type default)
+		)
+		(layer "Edge.Cuts")
+	)
 	(segment
 		(start 40.8 29.753)
@@
 		(net 17)
 	)
+	(segment
+		(start 313.5 57)
+		(end 313.5 78)
+		(width 0.25)
+		(layer "In4.Cu")
+		(net 18)
+	)
+	(segment
+		(start 313.5 78)
+		(end 315.5 80)
+		(width 0.25)
+		(layer "In4.Cu")
+		(net 18)
+	)
+	(segment
+		(start 315.5 80)
+		(end 315.5 99)
+		(width 0.25)
+		(layer "In4.Cu")
+		(net 18)
+	)
+	(segment
+		(start 315.5 99)
+		(end 315.5 118)
+		(width 0.25)
+		(layer "In4.Cu")
+		(net 18)
+	)
 	(via micro
 		(at 315.5 118)
@@
 	)
 	(segment
-		(start 315.7025 98.7975)
-		(end 315.5 99)
+		(start 315.7025 79.7975)
+		(end 315.7025 77.235)
 		(width 0.25)
 		(layer "B.Cu")
@@
 	)
 	(segment
-		(start 315.7025 79.7975)
-		(end 315.7025 77.235)
+		(start 315.7025 98.7975)
+		(end 315.5 99)
 		(width 0.25)
 		(layer "B.Cu")
@@
 	)
 	(segment
-		(start 315.5 80)
-		(end 315.7025 79.7975)
+		(start 315.7025 96.285)
+		(end 315.7025 98.7975)
 		(width 0.25)
 		(layer "B.Cu")
@@
 	)
 	(segment
-		(start 315.7025 96.285)
-		(end 315.7025 98.7975)
+		(start 315.5 80)
+		(end 315.7025 79.7975)
 		(width 0.25)
 		(layer "B.Cu")
@@
 	)
 	(segment
-		(start 293.3511 67.7)
-		(end 297 71.3489)
-		(width 0.25)
-		(layer "F.Cu")
-		(net 143)
-	)
-	(segment
-		(start 266.6489 71.3489)
-		(end 286.7511 71.3489)
-		(width 0.25)
-		(layer "F.Cu")
-		(net 143)
-	)
-	(segment
 		(start 286.7511 71.3489)
 		(end 287.1 71)
@@
 	)
 	(segment
-		(start 292 67.7)
-		(end 293.3511 67.7)
+		(start 266.6489 71.3489)
+		(end 286.7511 71.3489)
 		(width 0.25)
 		(layer "F.Cu")
@@
 	)
 	(segment
-		(start 320.6511 71.3489)
-		(end 321 71)
-		(width 0.25)
-		(layer "F.Cu")
-		(net 143)
-	)
-	(segment
-		(start 297 71.3489)
-		(end 320.6511 71.3489)
-		(width 0.25)
-		(layer "F.Cu")
-		(net 143)
-	)
-	(segment
 		(start 336.7 67.7)
 		(end 340 71)
@@
 	)
 	(segment
+		(start 320.6511 71.3489)
+		(end 321 71)
+		(width 0.25)
+		(layer "F.Cu")
+		(net 211)
+	)
+	(segment
+		(start 292 67.7)
+		(end 293.3511 67.7)
+		(width 0.25)
+		(layer "F.Cu")
+		(net 211)
+	)
+	(segment
+		(start 293.3511 67.7)
+		(end 297 71.3489)
+		(width 0.25)
+		(layer "F.Cu")
+		(net 211)
+	)
+	(segment
+		(start 297 71.3489)
+		(end 320.6511 71.3489)
+		(width 0.25)
+		(layer "F.Cu")
+		(net 211)
+	)
+	(segment
 		(start 378.1 71)
 		(end 367.3 71)
 		(width 0.25)
 		(layer "F.Cu")
-		(net 212)
+		(net 213)
 	)
 	(segment
@@
 		(width 0.25)
 		(layer "F.Cu")
-		(net 212)
+		(net 213)
 	)
 	(zone

Commit message: update
Parts:
- added J1: USB_C_Receptacle_USB2.0_16P, Connector_USB:USB_C_Receptacle_GCT_USB4110, B.Cu at (52.0, 22.5)
- added R1: 5K1, Resistor_SMD:R_2010_5025Metric_Pad1.40x2.65mm_HandSolder, B.Cu at (47.0, 30.9)
- added R2: 5K1, Resistor_SMD:R_2010_5025Metric_Pad1.40x2.65mm_HandSolder, B.Cu at (57.0, 30.9)
- added SW1: 3983, kb2040:SW_3983_ADA, B.Cu at (384.0, 37.2)
- added U1: RP2040_Stamp, kb2040:RP2xxx_Stamp_SMD, B.Cu at (359.5, 37.5)
Routing:
- net GND: track 0.00 -> 403.4 mm, vias 0 -> 2
- net Net-(U1-USB_D+): track 0.00 -> 374.5 mm, vias 0 -> 2
- net Net-(U1-USB_D-): track 0.00 -> 364.3 mm, vias 0 -> 2
- net col0: track 113.6 -> 464.4 mm
- net col1: track 84.5 -> 434.7 mm, vias 2 -> 4
- net Net-(U1-5V): track 0.00 -> 347.2 mm, vias 0 -> 2
- net col2: track 116.4 -> 424.5 mm
- net col3: track 136.9 -> 423.9 mm
- net col4: track 110.4 -> 376.5 mm
- net col6: track 99.1 -> 350.6 mm, vias 5 -> 7
- net col5: track 110.5 -> 355.7 mm
- net col7: track 115.6 -> 326.7 mm
- net col8: track 113.6 -> 303.0 mm
- net col9: track 113.5 -> 281.5 mm
- net col10: track 135.7 -> 282.4 mm
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Other:
- board text added: "(C) J. Westley 2024 No Arrows Keyboard - Designed for and with Dad Christmas '24"
