File: layout-pcb/keyboard.kicad_pcb (KiCad board)
At the start: 6 copper layers, 374.7 x 131.8 mm, 281 parts, among them J1 USB_C_Receptacle_USB2.0_16P, SW1 3983, U1 RP2040_Stamp

Commit message: LED placemnet #D hotswap and switch
Parts:
- D1: footprint LED_SMD:LED_WS2812B_PLCC4_5.0x5.0mm_P3.2mm -> WS2812-2020:LED_WS2812-2020
- J1: footprint Connector_USB:USB_C_Receptacle_GCT_USB4110 -> Connector_USB:USB_C_Receptacle_G-Switch_GT-USB-7010ASV
- K_ESC1: value KEYSW -> ESC
- R1, R2: footprint Resistor_SMD:R_2010_5025Metric_Pad1.40x2.65mm_HandSolder -> Resistor_SMD:R_01005_0402Metric_Pad0.57x0.30mm_HandSolder
- SW1: value 3983 -> SW_Push; footprint kb2040:SW_3983_ADA -> Button_Switch_THT:SW_PUSH_6mm
- moved R1 331.5 mm to (378.5, 28.5), turned to -90 degrees
- moved J1 327.8 mm to (379.8, 22.6)
- moved R2 323.0 mm to (380.0, 28.5), turned to -90 degrees
- moved D92 20.1 mm to (325.0, 31.4)
- moved D94 11.6 mm to (379.6, 31.4)
- moved SW1 7.53 mm to (391.5, 36.5), turned to 180 degrees
- moved D14 6.89 mm to (26.5, 71.5)
- moved U1 5.00 mm to (354.5, 37.5)
- moved D93 3.78 mm to (352.3, 31.4)
- moved D15 2.97 mm to (50.0, 71.5)
- moved D1 1.71 mm to (32.5, 42.5)
- moved D85 1.65 mm to (154.1, 147.5)
- moved D16 0.85 mm to (70.0, 70.0)
Connections:
- J1 pad A6: GND -> Net-(U1-USB_D+)
- J1 pad B6: GND -> Net-(U1-USB_D+)
- SW1 pad 1: Net-(U1-BOOTSEL) -> GND
- SW1 pad 2: GND -> Net-(U1-BOOTSEL)
- U1 pad 36: GND -> Net-(U1-USB_D+)
Routing:
- net GND: track 783.0 -> 41.0 mm, vias 2 -> 0
- net Net-(U1-USB_D-): track 364.3 -> 29.7 mm
- net Net-(U1-5V): track 347.2 -> 25.4 mm
- net Net-(U1-USB_D+): track 0.00 -> 30.0 mm
- net Net-(D92-DOUT): track 17.3 -> 33.5 mm
- net Net-(D93-DOUT): track 18.4 -> 33.5 mm
- net Net-(J1-CC1): track 9.67 -> 1.89 mm
- net Net-(J1-CC2): track 9.46 -> 2.88 mm
- net col5: track 355.7 -> 349.1 mm
- net col6: track 350.6 -> 344.1 mm
- net Net-(D14-DIN): track 15.5 -> 21.7 mm
- net col4: track 376.5 -> 370.4 mm
- net col9: track 281.5 -> 275.7 mm
- net 14p2-32p4: track 21.2 -> 26.9 mm
- net col7: track 326.7 -> 321.0 mm
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Other:
- board text added: "(C) J. Westley 2024 No Arrows Keybaord Desinged for ZMK & Dad github.com/Frank-08/zmk-config"
- board text added: "5K1"

Commit message: LED Pwr + Gnd moved to top LED planes removed
Parts:
- added TP1: LED_PWR, TestPoint:TestPoint_Pad_D3.0mm, B.Cu at (293.5, 39.5)
- added TP2: LED_GND, TestPoint:TestPoint_Pad_D3.0mm, B.Cu at (300.0, 39.5)
- added TP3: +5V, TestPoint:TestPoint_Pad_D3.0mm, B.Cu at (307.0, 39.0)
- added TP4: GND, TestPoint:TestPoint_Pad_D3.0mm, B.Cu at (377.0, 38.0)
- D1: footprint WS2812-2020:LED_WS2812-2020 -> LED_SMD:LED_WS2812B-Mini_PLCC4_3.5x3.5mm
- D10, D11, D12, D13, D14, D15, D16, D17, D18, D19, D2, D20, D21, D22, D23, D24, D25, D26, D27, D28, D29, D3, D30, D31, D32, D33, D34, D35, D36, D37, D38, D39, D4, D40, D41, D42, D43, D44, D45, D46, D47, D48, D49, D5, D50, D51, D52, D53, D54, D55, D56, D57, D58, D59, D6, D60, D61, D62, D63, D64, D65, D66, D67, D68, D69, D7, D70, D71, D72, D73, D74, D75, D76, D77, D78, D79, D8, D80, D81, D82, D83, D84, D85, D86, D87, D88, D89, D9, D90, D91, D92, D93, D94: footprint LED_SMD:LED_WS2812B_PLCC4_5.0x5.0mm_P3.2mm -> LED_SMD:LED_WS2812B-Mini_PLCC4_3.5x3.5mm
- R1, R2: footprint Resistor_SMD:R_01005_0402Metric_Pad0.57x0.30mm_HandSolder -> Resistor_SMD:R_0603_1608Metric_Pad0.98x0.95mm_HandSolder
- moved R2 6.08 mm to (386.0, 27.5)
- moved D14 5.96 mm to (32.4, 70.4)
- moved R1 5.10 mm to (373.5, 27.5)
- moved D29 2.95 mm to (339.6, 70.2)
- moved D19 2.15 mm to (127.5, 71.5)
- moved D49 2.15 mm to (380.5, 99.7)
- moved D81 2.15 mm to (380.1, 138.0)
- moved D82 2.15 mm to (35.0, 148.0)
- moved D83 2.15 mm to (58.5, 148.0)
- moved D84 2.15 mm to (82.5, 148.0)
- moved D86 2.15 mm to (225.6, 148.0)
- moved D87 2.15 mm to (249.6, 148.0)
- moved D88 2.15 mm to (273.1, 148.0)
- moved D89 2.15 mm to (297.1, 148.0)
- moved D90 2.15 mm to (333.1, 148.0)
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Connections:
- net Net-(U1-5V) renamed +5V 
Routing:
- net LED_PWR: track 169.5 -> 2270.4 mm, vias 94 -> 9
- net LED_GND: track 205.0 -> 2278.0 mm, vias 94 -> 14
- net +5V : track 25.4 -> 130.7 mm, vias 2 -> 5
- net 31p4 - 13p2: track 96.3 -> 109.2 mm
- net Net-(U1-BOOTSEL): track 16.1 -> 27.6 mm
- net GND: track 41.0 -> 49.7 mm
- net Net-(D14-DIN): track 21.7 -> 15.6 mm
- net Net-(J1-CC1): track 1.89 -> 7.90 mm
- net Net-(J1-CC2): track 2.88 -> 7.42 mm
- net col17: track 122.1 -> 117.7 mm, vias 5 -> 6
- net Net-(D29-DIN): track 15.6 -> 19.5 mm
- net Net-(D72-DOUT): track 26.9 -> 24.0 mm
- net Net-(D37-DOUT): track 24.9 -> 22.0 mm
- net Net-(D38-DOUT): track 26.4 -> 23.5 mm
- net Net-(D40-DOUT): track 25.9 -> 23.0 mm
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- removed copper zone on In2.Cu, net LED_GND
- removed copper zone on In1.Cu, net LED_PWR
Other:
- copper layers 6 -> 4

Commit message: Add JLCx3
Other:
- board text added: "JLCJLCJLCJLC"
Changed lines of the file:
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@@
 		(layer "Edge.Cuts")
+	)
+	(gr_text "JLCJLCJLCJLC"
+		(at 360 30 0)
+		(layer "B.SilkS")
+		(effects
+			(font
+				(size 1 1)
+				(thickness 0.15)
+			)
+			(justify left bottom mirror)
+		)
 	)
 	(gr_text "5K1"

Commit message: gen updates /w Dad
Parts:
- removed TP1: LED_PWR, TestPoint:TestPoint_Pad_D3.0mm
- removed TP2: LED_GND, TestPoint:TestPoint_Pad_D3.0mm
Connections:
- D1 pad 1: LED_PWR -> +5V 
- D10 pad 1: LED_PWR -> +5V 
- D11 pad 1: LED_PWR -> +5V 
- D12 pad 1: LED_PWR -> +5V 
- D13 pad 1: LED_PWR -> +5V 
- D14 pad 1: LED_PWR -> +5V 
- D15 pad 1: LED_PWR -> +5V 
- D16 pad 1: LED_PWR -> +5V 
- D17 pad 1: LED_PWR -> +5V 
- D18 pad 1: LED_PWR -> +5V 
- D19 pad 1: LED_PWR -> +5V 
- D2 pad 1: LED_PWR -> +5V 
- D20 pad 1: LED_PWR -> +5V 
- D21 pad 1: LED_PWR -> +5V 
- D22 pad 1: LED_PWR -> +5V 
- D23 pad 1: LED_PWR -> +5V 
- D24 pad 1: LED_PWR -> +5V 
- D25 pad 1: LED_PWR -> +5V 
- D26 pad 1: LED_PWR -> +5V 
- D27 pad 1: LED_PWR -> +5V 
- D28 pad 1: LED_PWR -> +5V 
- D29 pad 1: LED_PWR -> +5V 
- D3 pad 1: LED_PWR -> +5V 
- D30 pad 1: LED_PWR -> +5V 
- D31 pad 1: LED_PWR -> +5V 
- D4 pad 1: LED_PWR -> +5V 
- D5 pad 1: LED_PWR -> +5V 
- D6 pad 1: LED_PWR -> +5V 
- D7 pad 1: LED_PWR -> +5V 
- D8 pad 1: LED_PWR -> +5V 
- D9 pad 1: LED_PWR -> +5V 
- D92 pad 1: LED_PWR -> +5V 
- D93 pad 1: LED_PWR -> +5V 
- D94 pad 1: LED_PWR -> +5V 
Routing:
- net +5V : track 130.7 -> 920.6 mm, vias 5 -> 7
- net LED_PWR: track 2270.4 -> 1494.2 mm, vias 9 -> 7
