File: layout-pcb/_autosave-keyboard.kicad_pcb (KiCad board)
At the start: 6 copper layers, 374.7 x 131.8 mm, 281 parts, among them J1 USB_C_Receptacle_USB2.0_16P, SW1 3983, U1 RP2040_Stamp

Commit message: update
Parts:
- K_13: value KEYSW -> ~
- K_14: value KEYSW -> 1
- K_15: value KEYSW -> 2
- K_16: value KEYSW -> 3
- K_17: value KEYSW -> 4
- K_18: value KEYSW -> 5
- K_19: value KEYSW -> 6
- K_20: value KEYSW -> 7
- K_21: value KEYSW -> 8
- K_22: value KEYSW -> 9
- K_23: value KEYSW -> 0
- K_24: value KEYSW -> -
- K_25: value KEYSW -> =
- K_26: value KEYSW2 -> Backspace
- K_27: value KEYSW -> Num Lock
- K_28: value KEYSW -> Num Divide
- K_29: value KEYSW -> Num Multi
- K_30: value KEYSW -> Num Sub
- K_31: value KEYSW1.5 -> Tab
- K_32: value KEYSW -> Q
- K_33: value KEYSW -> W
- K_34: value KEYSW -> E
- K_35: value KEYSW -> R
- K_36: value KEYSW -> T
- K_37: value KEYSW -> Y
- K_38: value KEYSW -> U
- K_39: value KEYSW -> I
- K_40: value KEYSW -> O
- K_41: value KEYSW -> P
- K_42: value KEYSW -> [
- K_43: value KEYSW -> ]
- K_44: value KEYSW1.5 -> \
- K_45: value KEYSW -> Num 7
- K_46: value KEYSW -> Num 8
- K_47: value KEYSW -> Num 9
- K_48: value KEYSW -> Num Plus
- K_49: value KEYSW1.75 -> Caps Lock
- K_50: value KEYSW -> A
- K_51: value KEYSW -> S
- K_52: value KEYSW -> D
- K_53: value KEYSW -> F
- K_54: value KEYSW -> G
- K_55: value KEYSW -> H
- K_56: value KEYSW -> J
- K_57: value KEYSW -> K
- K_58: value KEYSW -> L
- K_59: value KEYSW -> ;
- K_60: value KEYSW -> '
- K_61: value KEYSW2.25 -> Enter
- K_62: value KEYSW -> Num 4
- K_63: value KEYSW -> Num 5
- K_64: value KEYSW -> Num 6
- K_65: value KEYSW2.25 -> Shift
- K_66: value KEYSW -> Z
- K_67: value KEYSW -> X
- K_68: value KEYSW -> C
- K_69: value KEYSW -> V
- K_70: value KEYSW -> B
- K_71: value KEYSW -> N
- K_72: value KEYSW -> M
- K_73: value KEYSW -> <
- K_74: value KEYSW -> >
- K_75: value KEYSW -> ?
- K_76: value KEYSW2.75 -> Shift
- K_77: value KEYSW -> Num 1
- K_78: value KEYSW -> Num 2
- K_79: value KEYSW -> Num 3
- K_80: value KEYSW -> Num Enter
- K_81, K_88: value KEYSW -> Ctrl
- K_82, K_86: value KEYSW -> Apple
- K_83, K_85: value KEYSW -> Alt
- K_84: value KEYSW6.25 -> Where Astronauts Hang Out
- K_87: value KEYSW -> Function
- K_89: value KEYSW2 -> Num 0
- K_90: value KEYSW -> Num .
- K_ESC1: value KEYSW -> ESC
- K_F1: value KEYSW -> F1
- K_F10: value KEYSW -> F10
- K_F11: value KEYSW -> F11
- K_F12: value KEYSW -> F12
- K_F2: value KEYSW -> F2
- K_F3: value KEYSW -> F3
- K_F4: value KEYSW -> F4
- K_F5: value KEYSW -> F5
- K_F6: value KEYSW -> F6
- K_F7: value KEYSW -> F7
- K_F8: value KEYSW -> F8
- K_F9: value KEYSW -> F9
- moved D92 20.1 mm to (325.0, 31.4)
- moved D94 11.6 mm to (379.6, 31.4)
- moved D93 3.78 mm to (352.3, 31.4)
Connections:
- J1 pad A6: GND -> Net-(U1-USB_D+)
- J1 pad B6: GND -> Net-(U1-USB_D+)
- U1 pad 36: GND -> Net-(U1-USB_D+)
Routing:
- net GND: track 783.0 -> 392.8 mm
- net Net-(U1-USB_D+): track 0.00 -> 374.5 mm
- net Net-(D92-DOUT): track 17.3 -> 33.5 mm
- net Net-(D93-DOUT): track 18.4 -> 33.5 mm
- net LED_PWR: track 168.5 -> 169.7 mm
Other:
- board text added: "(C) J. Westley 2024 No Arrows Keybaord Desinged for ZMK & Dad github.com/Frank-08/zmk-config"
