File: layout-pcb/_autosave-keyboard.kicad_sch (KiCad schematic)
At the start: 285 parts, among them J1 USB_C_Receptacle_USB2.0_16P, SW1 SW_Push, U1 RP2040_Stamp

Commit message: LED Pwr + Gnd moved to top LED planes removed
Connections:
- net LED_GND is gone; now on net GND: D1.3 (VSS), D10.3 (VSS), D11.3 (VSS), D12.3 (VSS), D13.3 (VSS), D14.3 (VSS), D15.3 (VSS), D16.3 (VSS), D17.3 (VSS), D18.3 (VSS), D19.3 (VSS), D2.3 (VSS), D20.3 (VSS), D21.3 (VSS), D22.3 (VSS), D23.3 (VSS), D24.3 (VSS), D25.3 (VSS), D26.3 (VSS), D27.3 (VSS), D28.3 (VSS), D29.3 (VSS), D3.3 (VSS), D30.3 (VSS), D31.3 (VSS), D32.3 (VSS), D33.3 (VSS), D34.3 (VSS), D35.3 (VSS), D36.3 (VSS), D37.3 (VSS), D38.3 (VSS), D39.3 (VSS), D4.3 (VSS), D40.3 (VSS), D41.3 (VSS), D42.3 (VSS), D43.3 (VSS), D44.3 (VSS), D45.3 (VSS), D46.3 (VSS), D47.3 (VSS), D48.3 (VSS), D49.3 (VSS), D5.3 (VSS), D50.3 (VSS), D51.3 (VSS), D52.3 (VSS), D53.3 (VSS), D54.3 (VSS), D55.3 (VSS), D56.3 (VSS), D57.3 (VSS), D58.3 (VSS), D59.3 (VSS), D6.3 (VSS), D60.3 (VSS), D61.3 (VSS), D62.3 (VSS), D63.3 (VSS), D64.3 (VSS), D65.3 (VSS), D66.3 (VSS), D67.3 (VSS), D68.3 (VSS), D69.3 (VSS), D7.3 (VSS), D70.3 (VSS), D71.3 (VSS), D72.3 (VSS), D73.3 (VSS), D74.3 (VSS), D75.3 (VSS), D76.3 (VSS), D77.3 (VSS), D78.3 (VSS), D79.3 (VSS), D8.3 (VSS), D80.3 (VSS), D81.3 (VSS), D82.3 (VSS), D83.3 (VSS), D84.3 (VSS), D85.3 (VSS), D86.3 (VSS), D87.3 (VSS), D88.3 (VSS), D89.3 (VSS), D9.3 (VSS), D90.3 (VSS), D91.3 (VSS), D92.3 (VSS), D93.3 (VSS), D94.3 (VSS), TP2.1
- net LED_PWR is gone; now on net +5V : D1.1 (VDD), D10.1 (VDD), D11.1 (VDD), D12.1 (VDD), D13.1 (VDD), D14.1 (VDD), D15.1 (VDD), D16.1 (VDD), D17.1 (VDD), D18.1 (VDD), D19.1 (VDD), D2.1 (VDD), D20.1 (VDD), D21.1 (VDD), D22.1 (VDD), D23.1 (VDD), D24.1 (VDD), D25.1 (VDD), D26.1 (VDD), D27.1 (VDD), D28.1 (VDD), D29.1 (VDD), D3.1 (VDD), D30.1 (VDD), D31.1 (VDD), D32.1 (VDD), D33.1 (VDD), D34.1 (VDD), D35.1 (VDD), D36.1 (VDD), D37.1 (VDD), D38.1 (VDD), D39.1 (VDD), D4.1 (VDD), D40.1 (VDD), D41.1 (VDD), D42.1 (VDD), D43.1 (VDD), D44.1 (VDD), D45.1 (VDD), D46.1 (VDD), D47.1 (VDD), D48.1 (VDD), D49.1 (VDD), D5.1 (VDD), D50.1 (VDD), D51.1 (VDD), D52.1 (VDD), D53.1 (VDD), D54.1 (VDD), D55.1 (VDD), D56.1 (VDD), D57.1 (VDD), D58.1 (VDD), D59.1 (VDD), D6.1 (VDD), D60.1 (VDD), D61.1 (VDD), D62.1 (VDD), D63.1 (VDD), D64.1 (VDD), D65.1 (VDD), D66.1 (VDD), D67.1 (VDD), D68.1 (VDD), D69.1 (VDD), D7.1 (VDD), D70.1 (VDD), D71.1 (VDD), D72.1 (VDD), D73.1 (VDD), D74.1 (VDD), D75.1 (VDD), D76.1 (VDD), D77.1 (VDD), D78.1 (VDD), D79.1 (VDD), D8.1 (VDD), D80.1 (VDD), D81.1 (VDD), D82.1 (VDD), D83.1 (VDD), D84.1 (VDD), D85.1 (VDD), D86.1 (VDD), D87.1 (VDD), D88.1 (VDD), D89.1 (VDD), D9.1 (VDD), D90.1 (VDD), D91.1 (VDD), D92.1 (VDD), D93.1 (VDD), D94.1 (VDD), TP1.1
Changed lines of the file:
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@@
 	)
 	(junction
+		(at 466.09 303.53)
+		(diameter 0)
+		(color 0 0 0 0)
+	)
+	(junction
 		(at 49.53 298.45)
 		(diameter 0)
@@
 	)
 	(junction
-		(at 63.5 254)
-		(diameter 0)
-		(color 0 0 0 0)
-	)
-	(junction
 		(at 375.92 151.13)
 		(diameter 0)
@@
 	(wire
 		(pts
+			(xy 466.09 307.34) (xy 466.09 303.53)
+		)
+		(stroke
+			(width 0)
+			(type default)
+		)
+	)
+	(wire
+		(pts
 			(xy 85.09 111.76) (xy 110.49 111.76)
 		)
@@
 	(wire
 		(pts
-			(xy 63.5 250.19) (xy 64.77 250.19)
-		)
-		(stroke
-			(width 0)
-			(type default)
-		)
-	)
-	(wire
-		(pts
 			(xy 111.76 402.59) (xy 111.76 401.32)
 		)
@@
 	(wire
 		(pts
-			(xy 63.5 254) (xy 63.5 250.19)
-		)
-		(stroke
-			(width 0)
-			(type default)
-		)
-	)
-	(wire
-		(pts
 			(xy 106.68 292.1) (xy 142.24 292.1)
 		)
@@
 		)
 	)
+	(global_label "LED_GND"
+		(shape input)
+		(at 466.09 307.34 270)
+		(fields_autoplaced yes)
+		(effects
+			(font
+				(size 1.27 1.27)
+			)
+			(justify right)
+		)
+		(property "Intersheetrefs" "${INTERSHEET_REFS}"
+			(at 466.09 317.9562 90)
+			(effects
+				(font
+					(size 1.27 1.27)
+				)
+				(justify right)
+				(hide yes)
+			)
+		)
+	)
 	(global_label "col12"
 		(shape input)
@@
 			(effects
 				(font
+					(size 1.27 1.27)
+				)
+				(justify left)
+				(hide yes)
+			)
+		)
+	)
+	(global_label "LED_PWR"
+		(shape input)
+		(at 462.28 229.87 90)
+		(fields_autoplaced yes)
+		(effects
+			(font
+				(size 1.27 1.27)
+			)
+			(justify left)
+		)
+		(property "Intersheetrefs" "${INTERSHEET_REFS}"
+			(at 462.28 219.1329 90)
+			(effects
+				(font
